File: Hardware/TXS0108 Breakout.brd (EAGLE design)
At the start: 27.9 x 12.7 mm, 61 parts, among them U1 TXS0108

Commit message: Design review revision
Parts:
- added U$33, U$47: (no value), output:#0
- added U$46, U$48: (no value), output:V0
- R1: value 10k -> 100k
- U$16: device output:#B5#0 -> output:#4#6
- U$17: device output:#B4#0 -> output:#5#6
- U$8: device output:#A4#0 -> output:#4#0
- U$9: device output:#A5#0 -> output:#5#0
- moved U$1 22.9 mm to (1.27, 6.60)
- moved U$2 22.9 mm to (1.27, 1.65)
- moved U$32 22.9 mm to (1.27, 11.0)
- moved U$34 22.9 mm to (1.27, 6.10)
- moved LOGO3 7.21 mm to (20.3, 6.35)
- moved U$17 5.18 mm to (16.5, 8.89)
- moved LOGO4 3.61 mm to (22.9, 6.35)
- moved U$43 2.79 mm to (19.3, 6.35)
- moved R1 2.69 mm to (20.3, 4.70), turned to 270 degrees
- moved U$19 2.54 mm to (8.89, 7.87)
- moved U$25 2.54 mm to (8.89, 5.08)
- moved U$27 2.54 mm to (14.0, 5.08)
- moved U$28 2.54 mm to (16.5, 4.95)
- moved U$38 2.54 mm to (16.5, 11.0)
- moved U$39 2.54 mm to (14.0, 11.0)
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Connections:
- removed net VCC_1: C1.1, C3.1, J1.11, U1.2
- removed net VCC_2: C2.1, C4.1, J2.10, U1.19
- new net VCCA: C1.1, C3.1, J1.10, U1.2
- new net VCCB: C2.1, C4.1, J2.9, U1.19
- net A1: now also J1.9; no longer J1.10
- net A2: now also J1.8; no longer J1.9
- net A3: now also J1.7; no longer J1.8
- net A4: now also J1.6; no longer J1.7
- net A5: now also J1.5; no longer J1.6
- net A6: now also J1.4; no longer J1.5
- net A7: now also J1.3; no longer J1.4
- net A8: now also J1.2; no longer J1.3
- net B1: now also J2.8; no longer J2.9
- net B2: now also J2.7; no longer J2.8
- net B3: now also J2.6; no longer J2.7
- net B4: now also J2.5; no longer J2.6
- net B5: now also J2.4; no longer J2.5
- net B6: now also J2.3; no longer J2.4
- net B7: now also J2.2; no longer J2.3
- net B8: now also J2.1; no longer J2.2
- net GND: now also J1.11, J2.10, U1.EPAD; no longer J1.2, J2.1
Routing:
- net VCC_2: track 13.8 -> 0.00 mm
- net VCC_1: track 13.8 -> 0.00 mm
- net VCCB: track 0.00 -> 12.8 mm, vias 0 -> 2
- net VCCA: track 0.00 -> 12.7 mm, vias 0 -> 2
- net OE: track 14.2 -> 11.2 mm
