File: Hardware/TXS0108 Breakout.brd (EAGLE design)
At the start: 27.9 x 12.7 mm, 65 parts, among them U1 TXS0108

Commit message: Add panelization v10
Other:
- board text added: "v10"
- board text removed: "v01"
Changed lines of the file:
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@@
 <drawing>
 <settings>
-<setting alwaysvectorfont="yes"/>
+<setting alwaysvectorfont="no"/>
 <setting verticaltext="up"/>
 </settings>
@@
 <wire x1="27.94" y1="12.7" x2="0" y2="12.7" width="0.2032" layer="20"/>
 <wire x1="0" y1="12.7" x2="0" y2="0" width="0.2032" layer="20"/>
-<text x="26.67" y="7.62" size="1.778" layer="16" font="vector" ratio="15" rot="SMR270" align="center">v01</text>
+<text x="26.67" y="7.62" size="1.778" layer="16" font="vector" ratio="15" rot="SMR270" align="center">v10</text>
 <text x="15.24" y="-8.89" size="1.778" layer="51" font="vector">Dryw Wade</text>
 <dimension x1="0" y1="12.7" x2="27.94" y2="12.7" x3="13.97" y3="16.51" textsize="1.778" textratio="15" layer="47" unit="inch"/>
