File: Hardware/TXS0108 Breakout.sch (EAGLE design)
At the start: 15 parts, among them U1 TXS0108

Commit message: Design review revision
Parts:
- R1: value 10k -> 100k; device SparkFun-Resistors:10KOHM-0603-1/10W-1% -> SparkFun-Resistors:100KOHM-0603-1/10W-1%
Connections:
- removed net VCC_1: C1.1, C3.1, J1.11, U1.VCCA
- removed net VCC_2: C2.1, C4.1, J2.10, U1.VCCB
- new net VCCA: C1.1, C3.1, J1.10, U1.VCCA
- new net VCCB: C2.1, C4.1, J2.9, U1.VCCB
- net A1: now also J1.9; no longer J1.10
- net A2: now also J1.8; no longer J1.9
- net A3: now also J1.7; no longer J1.8
- net A4: now also J1.6; no longer J1.7
- net A5: now also J1.5; no longer J1.6
- net A6: now also J1.4; no longer J1.5
- net A7: now also J1.3; no longer J1.4
- net A8: now also J1.2; no longer J1.3
- net B1: now also J2.8; no longer J2.9
- net B2: now also J2.7; no longer J2.8
- net B3: now also J2.6; no longer J2.7
- net B4: now also J2.5; no longer J2.6
- net B5: now also J2.4; no longer J2.5
- net B6: now also J2.3; no longer J2.4
- net B7: now also J2.2; no longer J2.3
- net B8: now also J2.1; no longer J2.2
- net GND: now also J1.11, J2.10, U1.EPAD; no longer J1.2, J2.1
Other:
- note added: "Must have VCCA <= VCCB!"
- note added: "OE voltage is referenced to VCCA"
- note added: "VCCA Range:"
- note added: "VCCB Range:"
- note removed: "OE voltage is based on VCC_1"
- note removed: "VCC_1 Range"
- note removed: "VCC_1 must be less than VCC_2!"
- note removed: "VCC_2 Range"
- moved on the sheet: J1, J2

Commit message: Add panelization v10
Other:
- note added: "v10"
- note removed: "v01"
Changed lines of the file:
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@@
 <wire x1="96.52" y1="124.46" x2="96.52" y2="132.08" width="0.2032" layer="97"/>
 <text x="166.624" y="11.43" size="2.54" layer="94" font="vector">Dryw Wade</text>
-<text x="239.268" y="7.366" size="2.54" layer="94" font="vector">v01</text>
+<text x="239.268" y="7.366" size="2.54" layer="94" font="vector">v10</text>
 </plain>
 <instances>
